File: PCB_V0.4.brd (EAGLE design)
At the start: 148.6 x 61.9 mm, 17 parts, among them J12 YK3310403000GCONN_YK331040XX0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, J13 61300411121, J8 61300311121

Commit message: Update files for 0.4 changes
Parts:
- added J1: 61300311121, 6130XX11121_61300311121:61300311121
- moved J13 15.3 mm to (129.5, 41.9)
- moved J12 2.54 mm to (147.3, 71.1)
Connections:
- new net N$1: J1.2, PD2.11
- net GND: now also J1.3
- net VIN+: now also J1.1
Routing:
- net N$1: track 0.00 -> 68.1 mm
- net GND: track 198.8 -> 255.4 mm
- net +5VCC1: track 59.2 -> 42.5 mm
- net GND1: track 59.3 -> 43.4 mm
- net +3.3VCC: track 54.7 -> 38.9 mm
- net VIN+: track 144.1 -> 153.9 mm
- net GND2: track 98.9 -> 100.7 mm
- net +5VCC: track 100.4 -> 101.6 mm
- net PA5: track 18.5 -> 17.5 mm
- net EN5+: track 58.9 -> 58.1 mm
Other:
- board text added: "**NOTE - GND IS ALREADY ROUTED FROM VIN-"
- board text added: "3: POWER DRIVERS, 0-50V"
- board text added: "5V-VR"
- board text added: "A+"
- board text added: "B+"
- board text added: "EN+"
- board text added: "EN1+"
- board text added: "EN2+"
- board text added: "GND-VR"
- board text added: "I/O"
- board text added: "M1:A+"
- board text added: "M1:B+"
- board text added: "M2:A+"
- board text added: "M2:B+"
- board text added: "M3:A+"
- board text added: "M3:B+"
- board text added: "MOTOR 1-7"
- board text added: "NULL"
- board text added: "SC1"
- board text added: "V0.4-MM"
- board text removed: "V0.3-MM"
